File: RvMeg_V2/RvMeg_V2.kicad_pcb (KiCad board)
At the start: 4 copper layers, 100.9 x 100 mm, 150 parts, among them J1 USB_B_Micro, J10 Encoder A, J11 Encoder B, J12 MPU6050, J13 ESC, J14 POWER, J15 Motor A, J16 Motor B, J2 Boot_Jumper, J3 J-Link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

Commit message: PCB Update
Parts:
- removed J2: Boot_Jumper, Connector_PinHeader_2.54mm:PinHeader_2x03_P2.54mm_Vertical
- added BOOT: SW_Push, Button_Switch_SMD:SW_Push_SPST_NO_Alps_SKRK, F.Cu at (113.1, 138.9)
- added C4: 0.1u, Capacitor_SMD:C_0805_2012Metric_Pad1.18x1.45mm_HandSolder, F.Cu at (112.0, 136.0)
- J14: value POWER -> VIN
- R2: moved to B.Cu
- moved R2 9.40 mm to (117.5, 136.9)
- moved R11 1.90 mm to (117.5, 140.7), turned to -90 degrees
- moved J3 0.38 mm to (127.3, 138.6)
- moved POWER 0.22 mm to (132.8, 138.8)
- moved RS12 0.06 mm to (186.7, 113.5)
- moved CONN_SEN_FRONT_I1 0.06 mm to (184.1, 112.3)
- moved CS7 0.06 mm to (187.1, 111.0)
- moved CS8 0.06 mm to (186.2, 111.0)
- moved LED_IR4 0.06 mm to (195.3, 111.0)
- moved MOSFET-N4 0.06 mm to (192.0, 113.2)
- moved Q6 0.06 mm to (188.8, 113.5)
- moved RS10 0.06 mm to (192.0, 110.6)
- moved RS8 0.06 mm to (197.3, 112.3)
Connections:
- R11 pad 1: Net-(J2-Pin_5) -> +3V3
- R11 pad 2: /BOOT_1 -> /BOOT_0
- R2 pad 1: /BOOT_0 -> /BOOT_1
- R2 pad 2: Net-(J2-Pin_2) -> GND
- U1 pad 10: /LEDs_1 -> /MENU
- U1 pad 39: /MENU -> /LEDs_1
Routing:
- net /MENU: track 122.6 -> 139.0 mm, vias 4 -> 2
- net /LEDs_1: track 83.2 -> 69.2 mm, vias 2 -> 6
- net /BOOT_0: track 30.3 -> 44.1 mm, vias 0 -> 1
- net +3V3: track 256.3 -> 247.6 mm
- net Net-(J2-Pin_2): track 3.08 -> 0.00 mm
- net /BOOT_1: track 4.81 -> 2.52 mm
- net Net-(J2-Pin_5): track 2.18 -> 0.00 mm
- net GND: track 12.3 -> 10.6 mm, vias 111 -> 112
- net /ENCODER_MotorB: track 75.2 -> 76.4 mm
- net /SWDIO: track 25.6 -> 26.2 mm
- net /SENSOR_CL_INPUT: track 104.3 -> 104.8 mm
Other:
- outline, holes or cut-outs redrawn
- board text added: "${REFERENCE}"
