File: RvMeg_V2/RvMeg_V2.kicad_sch (KiCad schematic)
At the start: 93 parts, among them J1 USB_B_Micro, J10 Encoder A, J11 Encoder B, J12 MPU6050, J13 ESC, J14 POWER, J15 Motor_A, J16 Motor_B, J2 Boot_Jumper, J3 J-Link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

Commit message: PCB Update
Parts:
- removed J2: Boot_Jumper, Connector_PinHeader_2.54mm:PinHeader_2x03_P2.54mm_Vertical, symbol Connector_Generic:Conn_02x03_Counter_Clockwise
- added BOOT1: SW_Push, Button_Switch_SMD:SW_Push_SPST_NO_Alps_SKRK, symbol EESTN5:SW_Push
- added C4: 0.1u, Capacitor_SMD:C_0805_2012Metric_Pad1.18x1.45mm_HandSolder, symbol Device:C
- added U7: MP1584_MODULE, MacroLib:MP1584_MODULE, symbol MacroLib:MP1584_MODULE
Connections:
- net +3V3: now also R11.1
- net BOOT_0: now also R11.2, BOOT1.2, C4.2; no longer R2.1
- net BOOT_1: now also R2.1; no longer R11.2
- net GND: now also R2.2, BOOT1.1, C4.1
- net LEDs_1: now also U1.39 (PB3); no longer U1.10 (PA0)
- net MENU: now also U1.10 (PA0); no longer U1.39 (PB3)
Other:
- moved on the sheet: C3, R11, R2, R3, RESET1
